File: 03 - Electrical Documentation/Wiring/Sample_wiring.sch (EAGLE design)
At the start: 3 parts

Commit message: Updated strain gauges and wiring diagram
Parts:
- added ENGINE_SPEED, ENGINE_TACHOMETER, LDS_BACKLEFT, LDS_BACKRIGHT, LDS_FRONTLEFT, LDS_FRONTRIGHT, PEDAL_BRAKE_POT, PEDAL_GAS_POT, TRANSFER_CASE_SPEED: SENSOR_1X3, wiring:SENSOR_1X3
- added IMU: SENSOR_SPI_2X3, wiring:SENSOR_SPI_2X3
- added U$10, U$11, U$15, U$19, U$20, U$6: WEATHERPACK_1X2_FEMALE, wiring:WEATHERPACK_1X2_FEMALE
- added U$12, U$18: BRAKELIGHT_SWITCH_HYDRAULIC, wiring:BRAKELIGHT_SWITCH_HYDRAULIC
- added U$13, U$16, U$17, U$5, U$7, U$8: WEATHERPACK_1X2_MALE, wiring:WEATHERPACK_1X2_MALE
- added U$14, U$21, U$22, U$24, U$25: MICROFIT_1X3_MALE, wiring:MICROFIT_1X3_MALE
- added U$23: MICROFIT_2X3_MALE, wiring:MICROFIT_2X3_MALE
- added U$26, U$27, U$28: SQUBA_1X4_MALE, wiring:SQUBA_1X4_MALE
- added U$29, U$30, U$31, U$32, U$33: MICROFIT_1X3_FEMALE, wiring:MICROFIT_1X3_FEMALE
- added U$4, U$9: SKIDOO_KILLSWITCH, wiring:SKIDOO_KILLSWITCH
- U$1: value MICROFIT_3X2_REC -> MICROFIT_1X3_MALE; device wiring:MICROFIT_3X2_REC -> wiring:MICROFIT_1X3_MALE
- U$2: value CMC_48PIN_PLUG -> CMC_48PIN_PLUG_PCB; device wiring:CMC_48PIN_PLUG -> wiring:CMC_48PIN_PLUG_PCB
Connections:
- removed net CMC: U$1.6
- new net B$1: IMU.1, IMU.2, IMU.3, IMU.4, IMU.5, IMU.6
- new net BRAKELIGHT+: U$16.1
- new net BRAKELIGHT-: U$16.2
- new net ENGINE_GND: U$7.2
- new net ENGINE_POS: U$7.1
- new net ENGINE_SPEED: U$27.BUS
- new net ENGINE_TACH: U$26.BUS
- new net IMU: U$23.BUS
- new net LDS_BL: U$14.BUS, U$31.BUS
- new net LDS_BR: U$22.BUS, U$32.BUS
- new net LDS_FL: U$1.BUS, U$29.BUS
- new net LDS_FR: U$21.BUS, U$30.BUS
- new net N$1: U$5.BUS, U$6.BUS
- new net N$10: U$11.BUS, U$7.BUS
- new net N$11: U$10.1, U$11.2, U$6.1
- new net N$12: U$13.BUS, U$15.BUS
- new net N$13: U$10.2, U$11.1, U$6.2
- new net N$14: U$13.1, U$18.P$2
- new net N$15: U$13.2, U$18.P$1
- new net N$16: U$17.BUS, U$19.BUS
- new net N$17: U$12.P$2, U$17.1
- new net N$18: U$12.P$1, U$17.2
- new net N$19: U$16.BUS, U$20.BUS
- new net N$20: U$15.1, U$19.1, U$20.2
- new net N$21: U$15.2, U$19.2, U$20.1
- new net N$22: LDS_BACKLEFT.3, U$14.3
- new net N$25: LDS_FRONTRIGHT.3, U$21.3
- new net N$26: LDS_FRONTRIGHT.2, U$21.2
- new net N$27: LDS_FRONTRIGHT.1, U$21.1
- new net N$28: LDS_BACKRIGHT.3, U$22.3
- new net N$29: LDS_BACKRIGHT.2, U$22.2
- new net N$30: LDS_BACKRIGHT.1, U$22.1
- new net N$31: PEDAL_BRAKE_POT.3, U$24.3
- new net N$32: PEDAL_BRAKE_POT.2, U$24.2
- new net N$33: PEDAL_BRAKE_POT.1, U$24.1
- new net N$34: PEDAL_GAS_POT.3, U$25.3
- new net N$35: PEDAL_GAS_POT.2, U$25.2
- new net N$36: PEDAL_GAS_POT.1, U$25.1
- new net N$37: ENGINE_TACHOMETER.3, U$26.3
- new net N$38: ENGINE_TACHOMETER.2, U$26.2
- new net N$39: ENGINE_TACHOMETER.1, U$26.1
- new net N$4: U$4.P$1, U$5.1
- new net N$40: U$25.BUS
- new net N$41: ENGINE_SPEED.3, U$27.3
- new net N$42: U$24.BUS
- new net N$43: ENGINE_SPEED.2, U$27.2
- new net N$44: ENGINE_SPEED.1, U$27.1
- new net N$45: TRANSFER_CASE_SPEED.3, U$28.3
- new net N$46: TRANSFER_CASE_SPEED.2, U$28.2
- new net N$47: TRANSFER_CASE_SPEED.1, U$28.1
- new net N$48: U$29.3, U$3.P$1
- new net N$49: U$29.2, U$3.P$2
- new net N$50: U$29.1, U$3.P$3
- new net N$51: U$3.P$4, U$30.3
- new net N$52: U$3.P$5, U$30.2
- new net N$53: U$3.P$6, U$30.1
- new net N$54: U$3.P$7, U$31.3
- new net N$55: U$3.P$8, U$31.2
- new net N$56: U$3.P$9, U$31.1
- new net N$57: U$3.P$10, U$32.3
- new net N$58: U$3.P$11, U$32.2
- new net N$59: U$3.P$12, U$32.1
- new net N$6: U$4.P$2, U$5.2
- new net N$60: U$3.P$61, U$33.3
- new net N$61: U$3.P$62, U$33.2
- new net N$62: U$3.P$63, U$33.1
- new net N$7: U$10.BUS, U$8.BUS
- new net N$8: U$8.1, U$9.P$1
- new net N$9: U$8.2, U$9.P$2
- new net TC_SPEED: U$28.BUS
- net N$2: now also LDS_FRONTLEFT.3
- net N$23: now also LDS_BACKLEFT.2, U$14.2; no longer U$1.4
- net N$24: now also LDS_BACKLEFT.1, U$14.1; no longer U$1.5
- net N$3: now also LDS_FRONTLEFT.2, U$1.2; no longer U$1.1
- net N$5: now also LDS_FRONTLEFT.1, U$1.1; no longer U$1.2
Other:
- note added: "Location: Top left chassis tube"

Commit message: updated wiring standards and docs
Parts:
- removed ENGINE_SPEED, ENGINE_TACHOMETER, TRANSFER_CASE_SPEED: SENSOR_1X3, wiring:SENSOR_1X3
- removed U$29, U$30, U$31, U$32, U$33: MICROFIT_1X3_FEMALE, wiring:MICROFIT_1X3_FEMALE
- added ENGINE_TACH_PCB: ENGINE_TACH_PCB, wiring:ENGINE_TACH_PCB
- added FREQ_SENSOR_ENGINE, FREQ_SENSOR_TRANSFER_CASE: SENSOR_1X3, wiring:SENSOR_1X3
Connections:
- removed net ENGINE_SPEED: U$27.BUS
- removed net ENGINE_TACH: U$26.BUS
- removed net IMU: U$23.BUS
- removed net LDS_BL: U$14.BUS, U$31.BUS
- removed net LDS_BR: U$22.BUS, U$32.BUS
- removed net LDS_FL: U$1.BUS, U$29.BUS
- removed net LDS_FR: U$21.BUS, U$30.BUS
- removed net N$10 (its old number): U$11.BUS, U$7.BUS
- removed net N$12 (its old number): U$13.BUS, U$15.BUS
- removed net N$16 (its old number): U$17.BUS, U$19.BUS
- removed net N$17 (its old number): U$12.P$2, U$17.1
- removed net N$18 (its old number): U$12.P$1, U$17.2
- removed net N$19 (its old number): U$16.BUS, U$20.BUS
- removed net N$40: U$25.BUS
- removed net N$41: ENGINE_SPEED.3, U$27.3
- removed net N$42: U$24.BUS
- removed net N$43: ENGINE_SPEED.2, U$27.2
- removed net N$44: ENGINE_SPEED.1, U$27.1
- removed net N$45: TRANSFER_CASE_SPEED.3, U$28.3
- removed net N$46: TRANSFER_CASE_SPEED.2, U$28.2
- removed net N$47: TRANSFER_CASE_SPEED.1, U$28.1
- removed net N$48: U$29.3, U$3.P$1
- removed net N$49: U$29.2, U$3.P$2
- removed net N$50: U$29.1, U$3.P$3
- removed net N$51: U$3.P$4, U$30.3
- removed net N$52: U$3.P$5, U$30.2
- removed net N$53: U$3.P$6, U$30.1
- removed net N$54: U$3.P$7, U$31.3
- removed net N$55: U$3.P$8, U$31.2
- removed net N$56: U$3.P$9, U$31.1
- removed net N$57: U$3.P$10, U$32.3
- removed net N$58: U$3.P$11, U$32.2
- removed net N$59: U$3.P$12, U$32.1
- removed net N$60: U$3.P$61, U$33.3
- removed net N$61: U$3.P$62, U$33.2
- removed net N$62: U$3.P$63, U$33.1
- removed net N$7 (its old number): U$10.BUS, U$8.BUS
- removed net N$8 (its old number): U$8.1, U$9.P$1
- removed net N$9 (its old number): U$8.2, U$9.P$2
- removed net TC_SPEED: U$28.BUS
- new net B$7: U$3.P$1, U$3.P$10, U$3.P$100, U$3.P$101, U$3.P$102, U$3.P$103, U$3.P$104, U$3.P$105, U$3.P$106, U$3.P$107, U$3.P$108, U$3.P$109, U$3.P$11, U$3.P$110, U$3.P$111, U$3.P$112, U$3.P$113, U$3.P$114, U$3.P$115, U$3.P$116, U$3.P$117, U$3.P$118, U$3.P$119, U$3.P$12, U$3.P$120, U$3.P$13, U$3.P$14, U$3.P$15, U$3.P$16, U$3.P$17, U$3.P$18, U$3.P$19, U$3.P$2, U$3.P$20, U$3.P$21, U$3.P$22, U$3.P$23, U$3.P$24, U$3.P$25, U$3.P$26, U$3.P$27, U$3.P$28, U$3.P$29, U$3.P$3, U$3.P$30, U$3.P$31, U$3.P$32, U$3.P$33, U$3.P$34, U$3.P$35, U$3.P$36, U$3.P$37, U$3.P$38, U$3.P$39, U$3.P$4, U$3.P$40, U$3.P$41, U$3.P$42, U$3.P$43, U$3.P$44, U$3.P$45, U$3.P$46, U$3.P$47, U$3.P$48, U$3.P$49, U$3.P$5, U$3.P$50, U$3.P$51, U$3.P$52, U$3.P$53, U$3.P$54, U$3.P$55, U$3.P$56, U$3.P$57, U$3.P$58, U$3.P$59, U$3.P$6, U$3.P$60, U$3.P$61, U$3.P$62, U$3.P$63, U$3.P$64, U$3.P$65, U$3.P$66, U$3.P$67, U$3.P$68, U$3.P$69, U$3.P$7, U$3.P$70, U$3.P$71, U$3.P$72, U$3.P$73, U$3.P$74, U$3.P$75, U$3.P$76, U$3.P$77, U$3.P$78, U$3.P$79, U$3.P$8, U$3.P$80, U$3.P$81, U$3.P$82, U$3.P$83, U$3.P$84, U$3.P$85, U$3.P$86, U$3.P$87, U$3.P$88, U$3.P$89, U$3.P$9, U$3.P$90, U$3.P$91, U$3.P$92, U$3.P$93, U$3.P$94, U$3.P$95, U$3.P$96, U$3.P$97, U$3.P$98, U$3.P$99
- new net N$2: U$4.P$1, U$5.2
- new net N$3: U$8.1, U$9.P$2
- new net N$31: FREQ_SENSOR_TRANSFER_CASE.1, U$28.1
- new net N$32: FREQ_SENSOR_TRANSFER_CASE.2, U$28.2
- new net N$33: FREQ_SENSOR_TRANSFER_CASE.3, U$28.3
- new net N$34: FREQ_SENSOR_ENGINE.1, U$27.1
- new net N$35: FREQ_SENSOR_ENGINE.2, U$27.2
- new net N$36: FREQ_SENSOR_ENGINE.3, U$27.3
- new net N$5: U$12.P$2, U$17.2
- new net SPARK_PLUG_WIRE: ENGINE_TACH_PCB.1
- net BRAKELIGHT+: now also U$16.2; no longer U$16.1
- net BRAKELIGHT-: now also U$16.1; no longer U$16.2
- net ENGINE_GND: now also ENGINE_TACH_PCB.2, U$7.1; no longer U$7.2
- net ENGINE_POS: now also U$7.2; no longer U$7.1
- net N$1: now also U$4.P$2, U$5.1; no longer U$5.BUS, U$6.BUS
- net N$20: now also U$19.2, U$20.1; no longer U$19.1, U$20.2
- net N$21: now also U$19.1, U$20.2; no longer U$19.2, U$20.1
- net N$37: now also ENGINE_TACH_PCB.6; no longer ENGINE_TACHOMETER.3
- net N$38: now also ENGINE_TACH_PCB.7; no longer ENGINE_TACHOMETER.2
- net N$39: now also ENGINE_TACH_PCB.8; no longer ENGINE_TACHOMETER.1
- net N$4: now also U$8.2, U$9.P$1; no longer U$4.P$1, U$5.1
- net N$6: now also U$12.P$1, U$17.1; no longer U$4.P$2, U$5.2
Other:
- note added: "Location: Above back left wheel"
- note added: "Location: Above back right wheel"
- note added: "Location: Above front left wheel"
- note added: "Location: Above front right wheel"
- note added: "Location: Along the spark plug wire"
- note added: "Location: Brake line"
- note added: "Location: By left elbow of driver"
- note added: "Location: Engine"
- note added: "Location: In front of right wing"
- note added: "Location: Transfer case cover"
- moved on the sheet: IMU, LDS_BACKLEFT, LDS_BACKRIGHT, LDS_FRONTLEFT, LDS_FRONTRIGHT, PEDAL_BRAKE_POT, PEDAL_GAS_POT

Commit message: updated car wiring
Parts:
- added BRAKE_PRESSURE_BACK, BRAKE_PRESSURE_FRONT: SENSOR_1X3, wiring:SENSOR_1X3
- added U$29: 3S 2200mAh, wiring:LIPO_BATT
- added U$30: 2S 1500mAh, wiring:LIPO_BATT
- added U$31: 2S, wiring:LIPO_BATT
- added U$32: WEATHERPACK_1X2_MALE, wiring:WEATHERPACK_1X2_MALE
- added U$33: MICROFIT_2X3_FEMALE, wiring:MICROFIT_2X3_FEMALE
- added U$34, U$35, U$36: SQUBA_1X4_FEMALE, wiring:SQUBA_1X4_FEMALE
- added U$37, U$38, U$39, U$40, U$41, U$42, U$43, U$44, U$45, U$46, U$49, U$50: MICROFIT_1X3_FEMALE, wiring:MICROFIT_1X3_FEMALE
- added U$47, U$48: METRIPACK_3PIN_FEMALE, wiring:METRIPACK_3PIN_FEMALE
Connections:
- removed net B$7: U$3.P$1, U$3.P$10, U$3.P$100, U$3.P$101, U$3.P$102, U$3.P$103, U$3.P$104, U$3.P$105, U$3.P$106, U$3.P$107, U$3.P$108, U$3.P$109, U$3.P$11, U$3.P$110, U$3.P$111, U$3.P$112, U$3.P$113, U$3.P$114, U$3.P$115, U$3.P$116, U$3.P$117, U$3.P$118, U$3.P$119, U$3.P$12, U$3.P$120, U$3.P$13, U$3.P$14, U$3.P$15, U$3.P$16, U$3.P$17, U$3.P$18, U$3.P$19, U$3.P$2, U$3.P$20, U$3.P$21, U$3.P$22, U$3.P$23, U$3.P$24, U$3.P$25, U$3.P$26, U$3.P$27, U$3.P$28, U$3.P$29, U$3.P$3, U$3.P$30, U$3.P$31, U$3.P$32, U$3.P$33, U$3.P$34, U$3.P$35, U$3.P$36, U$3.P$37, U$3.P$38, U$3.P$39, U$3.P$4, U$3.P$40, U$3.P$41, U$3.P$42, U$3.P$43, U$3.P$44, U$3.P$45, U$3.P$46, U$3.P$47, U$3.P$48, U$3.P$49, U$3.P$5, U$3.P$50, U$3.P$51, U$3.P$52, U$3.P$53, U$3.P$54, U$3.P$55, U$3.P$56, U$3.P$57, U$3.P$58, U$3.P$59, U$3.P$6, U$3.P$60, U$3.P$61, U$3.P$62, U$3.P$63, U$3.P$64, U$3.P$65, U$3.P$66, U$3.P$67, U$3.P$68, U$3.P$69, U$3.P$7, U$3.P$70, U$3.P$71, U$3.P$72, U$3.P$73, U$3.P$74, U$3.P$75, U$3.P$76, U$3.P$77, U$3.P$78, U$3.P$79, U$3.P$8, U$3.P$80, U$3.P$81, U$3.P$82, U$3.P$83, U$3.P$84, U$3.P$85, U$3.P$86, U$3.P$87, U$3.P$88, U$3.P$89, U$3.P$9, U$3.P$90, U$3.P$91, U$3.P$92, U$3.P$93, U$3.P$94, U$3.P$95, U$3.P$96, U$3.P$97, U$3.P$98, U$3.P$99
- new net N$40: U$20.1, U$32.2
- net B$1: now also U$23.1, U$23.2, U$23.3, U$23.4, U$23.5, U$23.6
- net N$20: now also U$32.1; no longer U$20.1
- net N$7: now also U$13.1; no longer U$13.2
- net N$8: now also U$13.2; no longer U$13.1
Other:
- note added: "Location: Below floorboard"
- moved on the sheet: ENGINE_TACH_PCB, FREQ_SENSOR_ENGINE, FREQ_SENSOR_TRANSFER_CASE

Commit message: Updated Brake Light Schematic
Connections:
- net N$20: now also U$15.2; no longer U$15.1
- net N$21: now also U$15.1; no longer U$15.2
Changed lines of the file:
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@@
 <setting verticaltext="up"/>
 </settings>
-<grid distance="0.1" unitdist="inch" unit="inch" style="lines" multiple="1" display="yes" altdistance="0.05" altunitdist="inch" altunit="inch"/>
+<grid distance="0.1" unitdist="inch" unit="inch" style="lines" multiple="1" display="no" altdistance="0.01" altunitdist="inch" altunit="inch"/>
 <layers>
 <layer number="1" name="Top" color="4" fill="1" visible="no" active="no"/>
@@
 <instance part="U$12" gate="G$1" x="15.24" y="-142.24" smashed="yes" rot="R90" grouprefs="BRAKELIGHT_SWITCHES"/>
 <instance part="U$13" gate="G$1" x="73.66" y="-142.24" smashed="yes" rot="R90" grouprefs="BRAKELIGHT_SWITCHES"/>
-<instance part="U$15" gate="G$1" x="88.9" y="-142.24" smashed="yes" rot="R90" grouprefs="BRAKELIGHT_SWITCHES"/>
+<instance part="U$15" gate="G$1" x="93.98" y="-144.78" smashed="yes" rot="R270" grouprefs="BRAKELIGHT_SWITCHES"/>
 <instance part="U$16" gate="G$1" x="139.7" y="-144.78" smashed="yes" rot="R270" grouprefs="BRAKELIGHT_SWITCHES"/>
 <instance part="U$17" gate="G$1" x="22.86" y="-142.24" smashed="yes" rot="R90" grouprefs="BRAKELIGHT_SWITCHES"/>
@@
 <wire x1="63.5" y1="-132.08" x2="91.44" y2="-132.08" width="0.1524" layer="91" grouprefs="BRAKELIGHT_SWITCHES"/>
 <wire x1="40.64" y1="-142.24" x2="40.64" y2="-132.08" width="0.1524" layer="91" grouprefs="BRAKELIGHT_SWITCHES"/>
-<pinref part="U$15" gate="G$1" pin="1"/>
-<wire x1="91.44" y1="-142.24" x2="91.44" y2="-132.08" width="0.1524" layer="91" grouprefs="BRAKELIGHT_SWITCHES"/>
 <pinref part="U$32" gate="G$1" pin="1"/>
 <wire x1="116.84" y1="-119.38" x2="116.84" y2="-111.76" width="0.1524" layer="91" grouprefs="BRAKELIGHT_SWITCHES"/>
@@
 <wire x1="63.5" y1="-111.76" x2="63.5" y2="-132.08" width="0.1524" layer="91" grouprefs="BRAKELIGHT_SWITCHES"/>
 <junction x="63.5" y="-132.08" grouprefs="BRAKELIGHT_SWITCHES"/>
+<pinref part="U$15" gate="G$1" pin="2"/>
+<wire x1="91.44" y1="-142.24" x2="91.44" y2="-132.08" width="0.1524" layer="91"/>
 </segment>
 </net>
 <net name="N$21" class="0">
 <segment>
+<pinref part="U$19" gate="G$1" pin="1"/>
 <wire x1="116.84" y1="-154.94" x2="91.44" y2="-154.94" width="0.1524" layer="91" grouprefs="BRAKELIGHT_SWITCHES"/>
-<pinref part="U$19" gate="G$1" pin="1"/>
 <wire x1="91.44" y1="-154.94" x2="40.64" y2="-154.94" width="0.1524" layer="91" grouprefs="BRAKELIGHT_SWITCHES"/>
 <wire x1="40.64" y1="-144.78" x2="40.64" y2="-154.94" width="0.1524" layer="91" grouprefs="BRAKELIGHT_SWITCHES"/>
-<pinref part="U$15" gate="G$1" pin="2"/>
-<wire x1="91.44" y1="-144.78" x2="91.44" y2="-154.94" width="0.1524" layer="91" grouprefs="BRAKELIGHT_SWITCHES"/>
-<junction x="91.44" y="-154.94" grouprefs="BRAKELIGHT_SWITCHES"/>
 <pinref part="U$20" gate="G$1" pin="2"/>
 <wire x1="116.84" y1="-144.78" x2="116.84" y2="-154.94" width="0.1524" layer="91" grouprefs="BRAKELIGHT_SWITCHES"/>
+<pinref part="U$15" gate="G$1" pin="1"/>
+<wire x1="91.44" y1="-144.78" x2="91.44" y2="-154.94" width="0.1524" layer="91"/>
+<junction x="91.44" y="-154.94"/>
 </segment>
 </net>
